File: index_keyboard.sch (KiCad schematic (older format))
At the start: 147 parts, among them CN1 MiniB USB, IC1 ATMEGA32U4-AU, J1 MX, K1 MX, M1 MX, P1 MX, Q1 MX, T1 MX, U1 MX, X1 MX, X3 16MHz, Y1 MX

Commit message: fixed diodes in schematic
Parts:
- gave numbers to parts that had none: 1
- renumbered C1 to C2, C2 to C3, C3 to C4, C7 to C5, C4 to C7, C5 to C8, D12 to D10, D13 to D11, D9 to D12, D10 to D13, D16 to D14, D17 to D15, D18 to D16, D19 to D17, D20 to D18, D21 to D19, D22 to D20, D23 to D21, D24 to D22, D25 to D23, D26 to D24, D27 to D25, D28 to D26, D30 to D27, D31 to D28, D32 to D29, D33 to D30, D34 to D31, D35 to D32, D36 to D33, D37 to D34, D38 to D35, D39 to D36, D40 to D37, D41 to D38, D42 to D39, D43 to D40, D44 to D41, D45 to D42, D46 to D43, D47 to D44, D48 to D45, D49 to D46, D50 to D47, D51 to D48, D52 to D49, D53 to D50, D54 to D51, D55 to D52, D56 to D53, D57 to D54, D58 to D55, D59 to D56, D60 to D57, D61 to D58, D62 to D59, D63 to D60, D14 to D61, D29 to D62, D15 to D63, D11 to D9, ISP6 to ISP1, L1 to L2, R3 to R2, R1 to R3, R2 to R4, R4 to R6, SJ2 to SJ1, SJ1 to SJ2, X3 to X2
Connections:
- wire segments 459 -> 350
Other:
- moved on the sheet: D1, D10, D11, D12, D13, D14, D15, D16, D17, D18, D19, D2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

Commit message: cleaned up some wire
Connections:
- wire segments 350 -> 360

Commit message: added pull up resistors to dip switches and increased dip switch count from 3 to 4 and removed the power led
Parts:
- removed 500mA1: L1, adafruit-R1206, symbol F_PTCFUSE
- removed PWR1: GREEN, adafruit-CHIPLED_0805, symbol LED_LED
- removed R6: 10K, adafruit-R0805, symbol R_R-US_
- removed SJ2: HWB, jumper-SJ, symbol SJ_SJ
- removed SW1: DIPS_03, symbol DIPS_03
- added R3, R4, R5: 3K, adafruit-R0805, symbol R_R-US_
- added SW1: DIPS_04, symbol DIPS_04
- R2: value 1K -> 3K
- renumbered D13 to D10, D9 to D11, D10 to D12, D11 to D13, D12 to D9, R3 to R6, R4 to R7, R5 to R8
Connections:
- wire segments 360 -> 367
